File: Synth.kicad_pcb (KiCad board)
At the start: 2 copper layers, 39.5 x 37.3 mm, 19 parts, among them J1 Screw_Terminal_01x02, J2 AudioJack2_Switch, Q1 2N3904, Q2 2N3904, Q3 2N3904, SW1 SW_Push

Commit message: added bom and fixed a resistor value in the schem - also added gerber
Parts:
- C1, C2, C3, C4: footprint Capacitor_SMD:CP_Elec_3x5.3 -> Capacitor_SMD:C_0603_1608Metric
Routing:
- net Net-(Q2-C): track 52.4 -> 53.8 mm
- net OscOut: track 49.7 -> 50.4 mm
- net Net-(Q1-C): track 9.04 -> 9.77 mm
- net AudioOut: track 3.91 -> 4.64 mm
- net 2: track 46.6 -> 47.3 mm
- net 1: track 15.2 -> 15.9 mm
