File: Synth.kicad_sch (KiCad schematic)
At the start: 19 parts, among them J1 Screw_Terminal_01x02, J2 AudioJack2_Switch, Q1 2N3904, Q2 2N3904, Q3 2N3904, SW1 SW_Push

Commit message: added bom and fixed a resistor value in the schem - also added gerber
Parts:
- C1, C2, C3, C4: footprint Capacitor_SMD:CP_Elec_3x5.3 -> Capacitor_SMD:C_0603_1608Metric
- R1: value R -> 1k
- R3: value 100k -> 10k
Changed lines of the file:
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@@
 			)
 		)
-		(property "Value" "100k"
+		(property "Value" "10k"
 			(at 147.32 82.5499 0)
 			(show_name no)
@@
 			)
 		)
-		(property "Footprint" "Capacitor_SMD:CP_Elec_3x5.3"
+		(property "Footprint" "Capacitor_SMD:C_0603_1608Metric"
 			(at 49.53 64.4652 0)
 			(hide yes)
@@
 			)
 		)
-		(property "Value" "R"
+		(property "Value" "1k"
 			(at 99.06 85.0899 0)
 			(show_name no)
@@
 			)
 		)
-		(property "Footprint" "Capacitor_SMD:CP_Elec_3x5.3"
+		(property "Footprint" "Capacitor_SMD:C_0603_1608Metric"
 			(at 143.8148 62.23 0)
 			(hide yes)
@@
 			)
 		)
-		(property "Footprint" "Capacitor_SMD:CP_Elec_3x5.3"
+		(property "Footprint" "Capacitor_SMD:C_0603_1608Metric"
 			(at 62.23 64.4652 0)
 			(hide yes)
@@
 			)
 		)
-		(property "Footprint" "Capacitor_SMD:CP_Elec_3x5.3"
+		(property "Footprint" "Capacitor_SMD:C_0603_1608Metric"
 			(at 173.99 61.2648 0)
 			(hide yes)
